File: PCB/SandyLPD_Base/SandyLPD_Base.kicad_pcb (KiCad board)
At the start: 2 copper layers, 270.8 x 100.7 mm, 295 parts, among them J1 Conn_02x02_Odd_Even, J10 Conn_01x10_Pin, J11 Conn_01x03, J12 Conn_01x01_Pin, J2 Conn_01x03, J3 Conn_01x01_Pin, J4 Conn_01x10_Pin, J5 USB_C_Receptacle_USB2.0, J6 USB_C_Receptacle_USB2.0, J7 USB_C_Receptacle_USB2.0, J8 USB_C_Receptacle_USB2.0, J9 Conn_02x02_Odd_Even, SW1 BOOT_ALT, SW2 RESET_ALT, SW3 SW_DIP_x04, SW4 BOOT_ALT, SW5 RESET_ALT, SW6 SW_DIP_x04, U1 NCP1117-3.3_SOT223, U2 NCP1117-3.3_SOT223, U3 RP2040, U4 W25Q128JVPIQ, U5 RP2040, U6 W25Q128JVPIQ, Y1 12MHz, Y2 12MHz

Commit message: スルーホールタップ位置確認。Base基板外形を左右へ拡大。
Parts:
- added Cutout1: 60_Outline, locallib:SandyLP_outline_Mid_Isolated_Area_gentle_corner, F.Cu at (-7.16, 46.2)
- added D1: D, locallib:D_SOD-123_Emphasized_Direction_Line, B.Cu at (-40.5, 35.5)
- added D2: D, locallib:D_SOD-123_Emphasized_Direction_Line, B.Cu at (-21.4, 35.5)
- added D3: D, locallib:D_SOD-123_Emphasized_Direction_Line, F.Cu at (-11.9, 35.5)
- added D4: D, locallib:D_SOD-123_Emphasized_Direction_Line, F.Cu at (-31.0, 35.5)
- added H1: MountingHole, locallib:MountingHole_2.2mm_M2_Pad_minimal, B.Cu at (-45.6, 27.7)
- added H2: MountingHole, locallib:MountingHole_2.2mm_M2_Pad_minimal, B.Cu at (-47.2, 43.3)
- added H3: MountingHole, locallib:MountingHole_2.2mm_M2_Pad_minimal, B.Cu at (-10.1, 27.7)
- added H4: MountingHole, locallib:MountingHole_2.2mm_M2_Pad_minimal, B.Cu at (-26.2, 36.1)
- added SW_BS1: SW_Push, locallib:Kailh_socket_ChocV2_for_Reverse_no_hole, B.Cu at (-35.7, 36.7)
- added SW_P1: SW_Push, locallib:Kailh_socket_ChocV2_small_#2pad_for_Reverse_no_hole, B.Cu at (-16.7, 36.7)
- added SW_Q1: SW_Push, locallib:Kailh_socket_ChocV2_for_Reverse, F.Cu at (-16.7, 36.7)
- added SW_TAB1: SW_Push, locallib:Kailh_socket_ChocV2_for_Reverse_narrow_#2pad, F.Cu at (-35.7, 36.7)
- added THC-0.8-x-2: MountingHole_2.2mm_M2_Pad_TopBottom, MountingHole:MountingHole_2.2mm_M2_Pad_TopBottom, F.Cu at (126.4, 35.3)
- added THC-0.8-x-2: MountingHole_2.2mm_M2_Pad_TopBottom, MountingHole:MountingHole_2.2mm_M2_Pad_TopBottom, F.Cu at (47.3, 45.5)
- added THC-0.8-x-2: MountingHole_2.2mm_M2_Pad_TopBottom, MountingHole:MountingHole_2.2mm_M2_Pad_TopBottom, F.Cu at (150.8, 52.6)
- added THC-0.8-x-2: MountingHole_2.2mm_M2_Pad_TopBottom, MountingHole:MountingHole_2.2mm_M2_Pad_TopBottom, F.Cu at (136.5, 74.6)
- added THC-0.8-x-2: MountingHole_2.2mm_M2_Pad_TopBottom, MountingHole:MountingHole_2.2mm_M2_Pad_TopBottom, F.Cu at (66.3, 74.6)
- added THC-0.8-x-2: MountingHole_2.2mm_M2_Pad_TopBottom, MountingHole:MountingHole_2.2mm_M2_Pad_TopBottom, F.Cu at (2.60, 77.6)
- added THC-0.8-x-2: MountingHole_2.2mm_M2_Pad_TopBottom, MountingHole:MountingHole_2.2mm_M2_Pad_TopBottom, F.Cu at (150.8, 90.7)
- added THC-0.8-x-2: MountingHole_2.2mm_M2_Pad_TopBottom, MountingHole:MountingHole_2.2mm_M2_Pad_TopBottom, F.Cu at (26.3, 52.7)
- added THC-0.8-x-2: MountingHole_2.2mm_M2_Pad_TopBottom, MountingHole:MountingHole_2.2mm_M2_Pad_TopBottom, F.Cu at (27.6, 111.5)
- added THC-0.8-x-2: MountingHole_2.2mm_M2_Pad_TopBottom, MountingHole:MountingHole_2.2mm_M2_Pad_TopBottom, F.Cu at (27.6, 35.3)
- added THC-0.8-x-2: MountingHole_2.2mm_M2_Pad_TopBottom, MountingHole:MountingHole_2.2mm_M2_Pad_TopBottom, F.Cu at (127.0, 55.6)
- added THC-0.8-x-2: MountingHole_2.2mm_M2_Pad_TopBottom, MountingHole:MountingHole_2.2mm_M2_Pad_TopBottom, F.Cu at (107.4, 35.3)
- added THC-0.8-x-2: MountingHole_2.2mm_M2_Pad_TopBottom, MountingHole:MountingHole_2.2mm_M2_Pad_TopBottom, F.Cu at (150.8, 110.9)
- added THC-0.8-x-2: MountingHole_2.2mm_M2_Pad_TopBottom, MountingHole:MountingHole_2.2mm_M2_Pad_TopBottom, F.Cu at (63.3, 35.3)
- added T_C0/C6: Conn_01x01, locallib:TestPoint_THTPad_D2.0mm_Drill1.0mm, B.Cu at (-26.2, 29.5)
- added T_R0: Conn_01x01, locallib:TestPoint_THTPad_D2.0mm_Drill1.0mm, B.Cu at (-45.3, 31.9)
- added T_R4: Conn_01x01, locallib:TestPoint_THTPad_D2.0mm_Drill1.0mm, B.Cu at (-45.3, 36.7)
- moved THC-0.8-x-2 90.0 mm to (150.8, 35.3)
- moved H_btm_7 8.95 mm to (159.8, 34.7)
- moved H_btm_8 8.42 mm to (159.2, 53.8)
- moved H_mid_19 5.36 mm to (150.2, 35.3)
Routing:
- net L_GPIO24: track 0.00 -> 99.4 mm
- net L_row0: track 0.00 -> 49.5 mm
- net L_col1: track 0.00 -> 49.3 mm
- net Net-(D1-A): track 0.00 -> 4.88 mm
- net Net-(D4-A): track 0.00 -> 4.88 mm
- net Net-(D2-A): track 0.00 -> 4.88 mm
- net Net-(D3-A): track 0.00 -> 4.24 mm
- net GND: vias 0 -> 18
Other:
- board size 270.8 x 100.7 mm -> 271.1 x 100.7 mm
- board text added: "ICON_Nut & Washer"
- board text added: "ICON_Screw_Long_Medium"
- board text added: "REF**"
- board text added: "Screw for SW-plate"
