File: PCB/SandyLPD_Plate_Base/SandyLPD_Plate_Base.kicad_sch (KiCad schematic)
At the start: 18 parts

Commit message: ロータリーエンコーダの穴をちょっと小さく。 #40
Parts:
- SW_13: footprint locallib:MX-Switch-Hole-for-RE(higher hole)-with-narrow-frame -> locallib:MX-Switch-Hole-for-RE(higher hole)-with-narrow-frame-gentle-corner
Changed lines of the file:
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@@
 			)
 		)
-		(property "Footprint" "locallib:MX-Switch-Hole-for-RE(higher hole)-with-narrow-frame"
+		(property "Footprint" "locallib:MX-Switch-Hole-for-RE(higher hole)-with-narrow-frame-gentle-corner"
 			(at 52.07 105.791 0)
 			(effects
