File: PCB/SandyLPD_Plate_BottomB/SandyLPD_Plate_BottomB.kicad_pcb (KiCad board)
At the start: 2 copper layers, 131 x 83 mm, 11 parts

Commit message: ネジの3Dモデル追加
Parts:
- H_btm_1, H_btm_3, H_btm_4: footprint locallib:MountingHole_2.2mm_M2_no_REF -> locallib:MountingHole_2.2mm_M2_no_REF_Plastic_L5mm; moved to F.Cu
- H_mid_1, H_mid_15, H_mid_19, H_mid_20, H_mid_21: footprint locallib:MountingHole_2.2mm_M2_no_REF -> locallib:MountingHole_2.2mm_M2_no_REF_Plastic_L5mm
- turned H_btm_1 to 0 degrees
- turned H_btm_3 to 0 degrees
- turned H_btm_4 to 0 degrees

Commit message: ネジの3Dモデルの向きを反転
Parts:
- H_btm_1, H_btm_3, H_btm_4, H_mid_1, H_mid_15, H_mid_19, H_mid_20, H_mid_21: moved to B.Cu
- turned H_btm_1 to 180 degrees
- turned H_btm_3 to 180 degrees
- turned H_btm_4 to 180 degrees
- turned H_mid_1 to 0 degrees
- turned H_mid_15 to 180 degrees
- turned H_mid_19 to 180 degrees
- turned H_mid_20 to 180 degrees
- turned H_mid_21 to 180 degrees
