File: PCB/SandyLPD_Mid-CNT/SandyLPD_Mid-CNT.kicad_sch (KiCad schematic)
At the start: 25 parts

Commit message: スイッチにネジ頭がかかるため、基板Baseと基板Mid-CNTを接続するネジ位置を調整。
Parts:
- H1, H2, H3, H4: footprint locallib:MountingHole_2.2-4.8mm_M2_Pad_minimal_for_Through-hole_tap -> locallib:MountingHole_2.2-4.8mm_M2_Pad_minimal_for_Through-hole_tap_L3mm
Changed lines of the file:
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@@
 			)
 		)
-		(property "Footprint" "locallib:MountingHole_2.2-4.8mm_M2_Pad_minimal_for_Through-hole_tap"
+		(property "Footprint" "locallib:MountingHole_2.2-4.8mm_M2_Pad_minimal_for_Through-hole_tap_L3mm"
 			(at 78.105 203.835 0)
 			(effects
@@
 			)
 		)
-		(property "Footprint" "locallib:MountingHole_2.2-4.8mm_M2_Pad_minimal_for_Through-hole_tap"
+		(property "Footprint" "locallib:MountingHole_2.2-4.8mm_M2_Pad_minimal_for_Through-hole_tap_L3mm"
 			(at 87.63 216.535 0)
 			(effects
@@
 			)
 		)
-		(property "Footprint" "locallib:MountingHole_2.2-4.8mm_M2_Pad_minimal_for_Through-hole_tap"
+		(property "Footprint" "locallib:MountingHole_2.2-4.8mm_M2_Pad_minimal_for_Through-hole_tap_L3mm"
 			(at 40.64 177.8 0)
 			(effects
@@
 			)
 		)
-		(property "Footprint" "locallib:MountingHole_2.2-4.8mm_M2_Pad_minimal_for_Through-hole_tap"
+		(property "Footprint" "locallib:MountingHole_2.2-4.8mm_M2_Pad_minimal_for_Through-hole_tap_L3mm"
 			(at 67.31 190.5 0)
 			(effects

Commit message: ネジ等の3Dモデル追加
Parts:
- H5: footprint locallib:MountingHole_M2_Through-hole_tap_THC-0.8-x-2 -> locallib:MountingHole_M2_Through-hole_tap_THC-0.8-1.0-2
Changed lines of the file:
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@@
 			)
 		)
-		(property "Footprint" "locallib:MountingHole_M2_Through-hole_tap_THC-0.8-x-2"
+		(property "Footprint" "locallib:MountingHole_M2_Through-hole_tap_THC-0.8-1.0-2"
 			(at 86.36 264.16 0)
 			(effects
