File: PCB/SandyLPD_Mid-ISO/SandyLPD_Mid-ISO.kicad_sch (KiCad schematic)
At the start: 17 parts

Commit message: スルーホールタップの接続先を変更・調整 #19
Parts:
- H1, H2, H3, H4: footprint locallib:MountingHole_2.2mm_M2_Pad_minimal -> locallib:MountingHole_2.2-4.8mm_M2_Pad_minimal_for_Through-hole_tap
- SW_TAB1: footprint locallib:Kailh_socket_ChocV2_for_Reverse_narrow_#2pad -> locallib:Kailh_socket_ChocV2_for_Reverse_narrow_#1_and_#2pad
Changed lines of the file:
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@@
 			)
 		)
-		(property "Footprint" "locallib:MountingHole_2.2mm_M2_Pad_minimal"
+		(property "Footprint" "locallib:MountingHole_2.2-4.8mm_M2_Pad_minimal_for_Through-hole_tap"
 			(at 66.675 111.125 0)
 			(effects
@@
 			)
 		)
-		(property "Footprint" "locallib:MountingHole_2.2mm_M2_Pad_minimal"
+		(property "Footprint" "locallib:MountingHole_2.2-4.8mm_M2_Pad_minimal_for_Through-hole_tap"
 			(at 66.675 121.285 0)
 			(effects
@@
 			)
 		)
-		(property "Footprint" "locallib:MountingHole_2.2mm_M2_Pad_minimal"
+		(property "Footprint" "locallib:MountingHole_2.2-4.8mm_M2_Pad_minimal_for_Through-hole_tap"
 			(at 38.735 111.125 0)
 			(effects
@@
 			)
 		)
-		(property "Footprint" "locallib:Kailh_socket_ChocV2_for_Reverse_narrow_#2pad"
+		(property "Footprint" "locallib:Kailh_socket_ChocV2_for_Reverse_narrow_#1_and_#2pad"
 			(at 43.18 45.72 0)
 			(effects
@@
 			)
 		)
-		(property "Footprint" "locallib:MountingHole_2.2mm_M2_Pad_minimal"
+		(property "Footprint" "locallib:MountingHole_2.2-4.8mm_M2_Pad_minimal_for_Through-hole_tap"
 			(at 38.735 121.285 0)
 			(effects

Commit message: ネジ等の3Dモデル追加
Parts:
- H1, H2, H3, H4: footprint locallib:MountingHole_2.2-4.8mm_M2_Pad_minimal_for_Through-hole_tap -> locallib:MountingHole_2.2-4.8mm_M2_Pad_minimal_for_Through-hole_tap_L3mm
- H5, H6: footprint locallib:MountingHole_M2_Through-hole_tap_THC-0.8-x-2 -> locallib:MountingHole_M2_Through-hole_tap_THC-0.8-1.0-2
Changed lines of the file:
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@@
 			)
 		)
-		(property "Footprint" "locallib:MountingHole_2.2-4.8mm_M2_Pad_minimal_for_Through-hole_tap"
+		(property "Footprint" "locallib:MountingHole_2.2-4.8mm_M2_Pad_minimal_for_Through-hole_tap_L3mm"
 			(at 66.675 111.125 0)
 			(effects
@@
 			)
 		)
-		(property "Footprint" "locallib:MountingHole_2.2-4.8mm_M2_Pad_minimal_for_Through-hole_tap"
+		(property "Footprint" "locallib:MountingHole_2.2-4.8mm_M2_Pad_minimal_for_Through-hole_tap_L3mm"
 			(at 66.675 121.285 0)
 			(effects
@@
 			)
 		)
-		(property "Footprint" "locallib:MountingHole_2.2-4.8mm_M2_Pad_minimal_for_Through-hole_tap"
+		(property "Footprint" "locallib:MountingHole_2.2-4.8mm_M2_Pad_minimal_for_Through-hole_tap_L3mm"
 			(at 38.735 111.125 0)
 			(effects
@@
 			)
 		)
-		(property "Footprint" "locallib:MountingHole_M2_Through-hole_tap_THC-0.8-x-2"
+		(property "Footprint" "locallib:MountingHole_M2_Through-hole_tap_THC-0.8-1.0-2"
 			(at 63.5 150.495 0)
 			(effects
@@
 			)
 		)
-		(property "Footprint" "locallib:MountingHole_M2_Through-hole_tap_THC-0.8-x-2"
+		(property "Footprint" "locallib:MountingHole_M2_Through-hole_tap_THC-0.8-1.0-2"
 			(at 38.1 162.56 0)
 			(effects
@@
 			)
 		)
-		(property "Footprint" "locallib:MountingHole_2.2-4.8mm_M2_Pad_minimal_for_Through-hole_tap"
+		(property "Footprint" "locallib:MountingHole_2.2-4.8mm_M2_Pad_minimal_for_Through-hole_tap_L3mm"
 			(at 38.735 121.285 0)
 			(effects
